Commit message: Atlas: remove all empty links (originally to put cameras into)

File: roboschool/models_robot/atlas_description/urdf/atlas_v4_with_multisense.urdf (robot description, URDF)
Before this commit: robot multisense_sl, 42 links, 41 joints
Links:
- removed link head_hokuyo_frame
- removed link head_imu_link
- removed link hokuyo_link
- removed link l_situational_awareness_camera_link
- removed link l_situational_awareness_camera_optical_frame
- removed link left_camera_frame
- removed link left_camera_optical_frame
- removed link r_situational_awareness_camera_link
- removed link r_situational_awareness_camera_optical_frame
- removed link right_camera_frame
- removed link right_camera_optical_frame
Joints:
- removed joint head_hokuyo_joint
- removed joint head_imu_joint
- removed joint hokuyo_joint
- removed joint l_situational_awareness_camera_joint
- removed joint l_situational_awareness_camera_optical_frame_joint
- removed joint left_camera_frame_joint
- removed joint left_camera_optical_frame_joint
- removed joint r_situational_awareness_camera_joint
- removed joint r_situational_awareness_camera_optical_frame_joint
- removed joint right_camera_frame_joint
- removed joint right_camera_optical_frame_joint

Commit message: Atlas experimental support

File: roboschool/models_robot/atlas_description/urdf/atlas_v4_with_multisense.urdf (robot description, URDF)
Before this commit: robot multisense_sl, 42 links, 41 joints
Links:
- removed link head_hokuyo_frame
- removed link head_imu_link
- removed link hokuyo_link
- removed link l_situational_awareness_camera_link
- removed link l_situational_awareness_camera_optical_frame
- removed link left_camera_frame
- removed link left_camera_optical_frame
- removed link r_situational_awareness_camera_link
- removed link r_situational_awareness_camera_optical_frame
- removed link right_camera_frame
- removed link right_camera_optical_frame
- link l_hand: mass 0.1 -> 1.0
- link r_hand: mass 0.1 -> 1.0
Joints:
- removed joint head_hokuyo_joint
- removed joint head_imu_joint
- removed joint hokuyo_joint
- removed joint l_situational_awareness_camera_joint
- removed joint l_situational_awareness_camera_optical_frame_joint
- removed joint left_camera_frame_joint
- removed joint left_camera_optical_frame_joint
- removed joint r_situational_awareness_camera_joint
- removed joint r_situational_awareness_camera_optical_frame_joint
- removed joint right_camera_frame_joint
- removed joint right_camera_optical_frame_joint
- joint l_leg_akx: limit lower=-0.8 upper=0.8 effort=360 velocity=12 -> lower=-0.8 upper=0.8 effort=45 velocity=12
- joint l_leg_aky: limit lower=-1 upper=0.7 effort=740 velocity=12 -> lower=-1 upper=0.7 effort=92 velocity=12
- joint r_leg_akx: limit lower=-0.8 upper=0.8 effort=360 velocity=12 -> lower=-0.8 upper=0.8 effort=45 velocity=12
- joint r_leg_aky: limit lower=-1 upper=0.7 effort=740 velocity=12 -> lower=-1 upper=0.7 effort=92 velocity=12
